File: hardware/inverter/cirBATTverter_1KWH.kicad_pcb (KiCad board)
At the start: 4 copper layers, 190.3 x 103.1 mm, 169 parts, among them J1 Conn_01x01, J2 Conn_01x01, J4 Conn_01x14, J5 Conn_01x29, J7 Conn_01x03, Q1 Q_NMOS_GDS, Q13 NPN, Q14 CID12N65D, Q15 CID12N65D, Q16 CID12N65D, Q17 CID12N65D, Q2 Q_NMOS_GDS, Q4 Q_NMOS_GDS, Q5 Q_NMOS_GDS, Q6 Q_NMOS_GDS, Q7 Q_NMOS_GDS, Q8 Q_NMOS_GDS, Q9 Q_NMOS_GDS, T1 Transformer_1P_2S, T4 CS4200V-01L, T5 Transformer_1P_1S, U1 Optocoupler_DC_PhotoNPN_AKEC, U2 TL431DBZ, U3 LM5013DDAR, U4 LM5013DDAR, U6 L7805

Commit message: Import supplied inverter corrections and document remaining design blockers
Connections:
- net /VFB renamed Net-(J4-Pin_5)
- J5 pad 13: GND2 -> unconnected-(J5-Pin_13-Pad13)
- J5 pad 15: /ISENSE3_P -> /ISENSE1_P
- J5 pad 17: /+15V -> unconnected-(J5-Pin_17-Pad17)
- J5 pad 22: GND2 -> unconnected-(J5-Pin_22-Pad22)
- J5 pad 26: unconnected-(J5-Pin_26-Pad26) -> /ISENSE1_N
- Q15 pad 12: /ISENSE3_P -> /ISENSE1_P
- R59 pad 1: /ISENSE3_P -> /ISENSE1_P
- U4 pad 10: GND2 -> (no net)
- U4 pad 11: GND2 -> (no net)
- U4 pad 12: GND2 -> (no net)
- U4 pad 13: GND2 -> (no net)
- U4 pad 14: GND2 -> (no net)
- U4 pad 15: GND2 -> (no net)
- U4 pad 16: GND2 -> (no net)
- U4 pad 17: GND2 -> (no net)
Routing:
- net /ISENSE1_P: track 103.1 -> 163.9 mm, vias 5 -> 9
- net /ISENSE3_P: track 58.4 -> 0.00 mm, vias 4 -> 0
- net /ISENSE1_N: track 117.4 -> 75.2 mm
- net /+12V: track 127.8 -> 109.0 mm
- net unconnected-(J5-Pin_22-Pad22): track 0.00 -> 2.10 mm, vias 0 -> 1
- net unconnected-(J5-Pin_13-Pad13): track 0.00 -> 1.80 mm, vias 0 -> 1
- net GND2: track 20.2 -> 19.3 mm, vias 212 -> 210
- removed copper zone on F.Cu, net /ISENSE3_P

Commit message: Import 17 October hardware corrections and document remaining review findings
Connections:
- J5 pad 15: /ISENSE1_P -> /ISENSE3_P
- Q15 pad 12: /ISENSE1_P -> /ISENSE3_P
- R35 pad 1: /400V -> /+400V
- R59 pad 1: /ISENSE1_P -> /ISENSE3_P
Routing:
- net /ISENSE1_P: track 163.9 -> 100.9 mm, vias 9 -> 5
- net /ISENSE3_P: track 0.00 -> 60.3 mm, vias 0 -> 4
- net /+400V: track 46.7 -> 64.0 mm, vias 53 -> 54
- net /+15V: track 193.5 -> 190.1 mm
- net unconnected-(J5-Pin_22-Pad22): track 2.10 -> 0.00 mm, vias 1 -> 0
- net unconnected-(J5-Pin_13-Pad13): track 1.80 -> 0.00 mm, vias 1 -> 0
- net /ISENSE1_N: track 75.2 -> 74.6 mm
- added copper zone on F.Cu, net /ISENSE3_P
