File: hardware/inverter/cirBATTverter_1KWH.kicad_pcb (KiCad board)
At the start: 4 copper layers, 190.3 x 103.1 mm, 169 parts, among them J1 Conn_01x01, J2 Conn_01x01, J4 Conn_01x14, J5 Conn_01x29, J7 Conn_01x03, Q1 Q_NMOS_GDS, Q13 NPN, Q14 CID12N65D, Q15 CID12N65D, Q16 CID12N65D, Q17 CID12N65D, Q2 Q_NMOS_GDS, Q4 Q_NMOS_GDS, Q5 Q_NMOS_GDS, Q6 Q_NMOS_GDS, Q7 Q_NMOS_GDS, Q8 Q_NMOS_GDS, Q9 Q_NMOS_GDS, T1 Transformer_1P_2S, T4 CS4200V-01L, T5 Transformer_1P_1S, U1 Optocoupler_DC_PhotoNPN_AKEC, U2 TL431DBZ, U3 LM5013DDAR, U4 LM5013DDAR, U6 L7805

Commit message: Import 20 October Q15 corrections and verify PCB production exports
Connections:
- C52 pad 2: /ISENSE1_P -> /ISENSE3_P
- C53 pad 2: /ISENSE1_P -> /ISENSE3_P
- Q15 pad 11: /ISENSE1_P -> /ISENSE3_P
- Q15 pad 7: /ISENSE1_P -> /ISENSE3_P
Routing:
- net /ISENSE1_P: track 100.9 -> 59.8 mm, vias 5 -> 4
- net /ISENSE3_P: track 60.3 -> 80.4 mm
