File: hardware/inverter/cirBATTverter_1KWH.kicad_sch (KiCad schematic)
At the start: 160 parts, among them J1 Conn_01x01, J2 Conn_01x01, J4 Conn_01x14, J5 Conn_01x29, J7 Conn_01x03, Q1 Q_NMOS_GDS, Q13 NPN, Q14 CID12N65D, Q15 CID12N65D, Q16 CID12N65D, Q17 CID12N65D, Q2 Q_NMOS_GDS, Q4 Q_NMOS_GDS, Q5 Q_NMOS_GDS, Q6 Q_NMOS_GDS, Q7 Q_NMOS_GDS, Q8 Q_NMOS_GDS, Q9 Q_NMOS_GDS, T1 Transformer_1P_2S, T4 CS4200V-01L, T5 Transformer_1P_1S, U1 Optocoupler_DC_PhotoNPN_AKEC, U2 TL431DBZ, U3 LM5013DDAR, U4 LM5013DDAR, U6 L7805

Commit message: Import supplied inverter corrections and document remaining design blockers
Connections:
- net ISENSE3_P is gone; now on net ISENSE1_P: J5.15 (Pin_15), Q15.12 (S), R59.1
- net +15V: no longer J5.17 (Pin_17)
- net GND2: no longer J5.13 (Pin_13), J5.22 (Pin_22)
- net ISENSE1_N: now also J5.26 (Pin_26)
- net VFB: no longer names the net of C7.1, J4.5 (Pin_5), R32.2, U1.3
- no-connect marks 8 -> 10
Other:
- moved on the sheet: R39, R50

Commit message: Import 17 October hardware corrections and document remaining review findings
Connections:
- net 400V is gone; now on net +400V: R35.1
- net ISENSE1_P: no longer J5.15 (Pin_15), Q15.12 (S), R59.1
- new net ISENSE3_P: J5.15 (Pin_15), Q15.12 (S), R59.1
Changed lines of the file:
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@@
 	)
 	(junction
+		(at 485.14 191.77)
+		(diameter 0)
+		(color 0 0 0 0)
+	)
+	(junction
 		(at 326.39 113.03)
 		(diameter 0)
@@
 	)
 	(junction
-		(at 485.14 191.77)
+		(at 419.1 191.77)
 		(diameter 0)
 		(color 0 0 0 0)
@@
 	)
 	(junction
-		(at 433.07 191.77)
-		(diameter 0)
-		(color 0 0 0 0)
-	)
-	(junction
 		(at 245.11 334.01)
 		(diameter 0)
@@
 	)
 	(junction
-		(at 419.1 191.77)
-		(diameter 0)
-		(color 0 0 0 0)
-	)
-	(junction
 		(at 96.52 142.24)
 		(diameter 0)
@@
 	(wire
 		(pts
-			(xy 433.07 191.77) (xy 485.14 191.77)
-		)
-		(stroke
-			(width 0)
-			(type default)
-		)
-	)
-	(wire
-		(pts
 			(xy 433.07 86.36) (xy 499.11 86.36)
 		)
@@
 	(wire
 		(pts
-			(xy 433.07 191.77) (xy 433.07 195.58)
-		)
-		(stroke
-			(width 0)
-			(type default)
-		)
-	)
-	(wire
-		(pts
 			(xy 240.03 119.38) (xy 240.03 116.84)
 		)
@@
 	(wire
 		(pts
-			(xy 419.1 191.77) (xy 433.07 191.77)
+			(xy 480.06 212.09) (xy 480.06 207.01)
 		)
 		(stroke
@@
 	(wire
 		(pts
-			(xy 480.06 212.09) (xy 480.06 207.01)
+			(xy 490.22 123.19) (xy 490.22 125.73)
 		)
 		(stroke
@@
 	(wire
 		(pts
-			(xy 490.22 123.19) (xy 490.22 125.73)
+			(xy 455.93 121.92) (xy 455.93 104.14)
 		)
 		(stroke
@@
 	(wire
 		(pts
-			(xy 455.93 121.92) (xy 455.93 104.14)
+			(xy 111.76 251.46) (xy 120.65 251.46)
 		)
 		(stroke
@@
 	(wire
 		(pts
-			(xy 111.76 251.46) (xy 120.65 251.46)
+			(xy 177.8 50.8) (xy 177.8 57.15)
 		)
 		(stroke
@@
 	(wire
 		(pts
-			(xy 177.8 50.8) (xy 177.8 57.15)
+			(xy 419.1 191.77) (xy 485.14 191.77)
 		)
 		(stroke
@@
 	(wire
 		(pts
-			(xy 433.07 177.8) (xy 433.07 191.77)
+			(xy 433.07 177.8) (xy 433.07 195.58)
 		)
 		(stroke
@@
 		)
 	)
-	(label "400V"
-		(at 176.53 245.11 0)
-		(effects
-			(font
-				(size 1.27 1.27)
-			)
-			(justify left bottom)
-		)
-	)
 	(label "OUT_HS1_N"
 		(at 501.65 146.05 0)
@@
 		(effects
 			(font
+				(size 1.27 1.27)
+			)
+			(justify left bottom)
+		)
+	)
+	(label "+400V"
+		(at 176.53 245.11 90)
+		(effects
+			(font

Commit message: Import 20 October Q15 corrections and verify PCB production exports
Connections:
- net ISENSE1_P: no longer C52.2, C53.2, Q15.11 (PGND), Q15.7 (SGND)
- net ISENSE3_P: now also C52.2, C53.2, Q15.11 (PGND), Q15.7 (SGND)
Changed lines of the file:
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@@
 	)
 	(junction
-		(at 485.14 191.77)
-		(diameter 0)
-		(color 0 0 0 0)
-	)
-	(junction
 		(at 326.39 113.03)
 		(diameter 0)
@@
 	)
 	(junction
-		(at 419.1 191.77)
-		(diameter 0)
-		(color 0 0 0 0)
-	)
-	(junction
 		(at 165.1 259.08)
 		(diameter 0)
@@
 	)
 	(junction
+		(at 419.1 191.77)
+		(diameter 0)
+		(color 0 0 0 0)
+	)
+	(junction
 		(at 433.07 86.36)
 		(diameter 0)
@@
 	)
 	(junction
+		(at 433.07 191.77)
+		(diameter 0)
+		(color 0 0 0 0)
+	)
+	(junction
 		(at 335.28 101.6)
 		(diameter 0)
@@
 	(wire
 		(pts
-			(xy 419.1 191.77) (xy 485.14 191.77)
+			(xy 140.97 265.43) (xy 132.08 265.43)
 		)
 		(stroke
@@
 	(wire
 		(pts
-			(xy 140.97 265.43) (xy 132.08 265.43)
+			(xy 154.94 251.46) (xy 161.29 251.46)
 		)
 		(stroke
@@
 	(wire
 		(pts
-			(xy 154.94 251.46) (xy 161.29 251.46)
+			(xy 496.57 125.73) (xy 494.03 125.73)
 		)
 		(stroke
@@
 	(wire
 		(pts
-			(xy 496.57 125.73) (xy 494.03 125.73)
+			(xy 104.14 349.25) (xy 104.14 337.82)
 		)
 		(stroke
@@
 	(wire
 		(pts
-			(xy 104.14 349.25) (xy 104.14 337.82)
+			(xy 523.24 237.49) (xy 523.24 240.03)
 		)
 		(stroke
@@
 	(wire
 		(pts
-			(xy 523.24 237.49) (xy 523.24 240.03)
+			(xy 146.05 97.79) (xy 148.59 97.79)
 		)
 		(stroke
@@
 	(wire
 		(pts
-			(xy 146.05 97.79) (xy 148.59 97.79)
+			(xy 433.07 191.77) (xy 433.07 195.58)
 		)
 		(stroke
@@
 	(wire
 		(pts
-			(xy 433.07 177.8) (xy 433.07 195.58)
+			(xy 433.07 177.8) (xy 433.07 191.77)
 		)
 		(stroke
@@
 		)
 		(stroke
+			(width 0)
+			(type default)
+		)
+	)
+	(wire
+		(pts
+			(xy 419.1 191.77) (xy 433.07 191.77)
+		)
+		(stroke
